File: UWB_ESP32S3_MainBoard_v2/UWB_ESP32S3_MainBoard_v2/UWB_ESP32S3_MainBoard_v2.kicad_pcb (KiCad board)
At the start: 2 copper layers, 90 x 90 mm, 39 parts, among them J1 ESP32_S3_2, J10 MP1584EN_IN, J11 MP1584EN_OUT, J12 MINI360_IN, J13 MINI360_OUT, J14 VBAT, J15 MOTOR_L, J16 MOTOR_R, J2 ESP32_S3_1, J3 BNO085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

Commit message: 배치중1
Parts:
- moved C5 252.8 mm to (-74.8, -20.2)
- moved C7 252.8 mm to (-74.8, -13.7)
- moved J10 252.8 mm to (-88.1, -21.2)
- moved J11 252.8 mm to (-83.5, -21.2)
- moved J12 252.8 mm to (-106.5, 22.6)
- moved J15 252.8 mm to (-98.0, -0.95)
- moved J16 252.8 mm to (-98.0, 8.40)
- moved J3 252.8 mm to (-75.3, -3.91)
- moved J4 252.8 mm to (-106.5, -21.2)
- moved J7 252.8 mm to (-92.7, -21.2)
- moved J8 252.8 mm to (-70.7, -3.91)
- moved R1 252.8 mm to (-84.9, 23.9)
- moved R2 252.8 mm to (-84.9, 26.9)
- moved R3 252.8 mm to (-84.9, 29.8)
- moved TP1 252.8 mm to (-79.2, -21.5)
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
Commit message: 배치 완료, 풋프린트 추가 등
Parts:
- added C12: 10uF_50V, Capacitor_SMD:C_0805_2012Metric_Pad1.18x1.45mm_HandSolder, F.Cu at (21.0, -41.0)
- added C13: 0.1uF_50V, Capacitor_SMD:C_0805_2012Metric_Pad1.18x1.45mm_HandSolder, F.Cu at (17.2, -41.0)
- added C14: 100uF_16V, Capacitor_THT:CP_Radial_D5.0mm_P2.00mm, F.Cu at (-19.8, -17.8)
- C11: value 470uF_16V -> 100uF_16V; footprint Capacitor_THT:CP_Radial_D8.0mm_P3.50mm -> Capacitor_THT:CP_Radial_D5.0mm_P2.00mm
- moved J9 145.1 mm to (39.2, 28.5), turned to -90 degrees
- moved J3 114.3 mm to (38.8, -11.4)
- moved C9 110.0 mm to (40.8, -19.2)
- moved C10 109.9 mm to (40.7, -16.2)
- moved J8 103.7 mm to (26.0, -41.5), turned to 90 degrees
- moved J13 103.7 mm to (-12.6, -30.0), turned to 90 degrees
- moved J12 101.1 mm to (-12.6, -14.8), turned to 90 degrees
- moved R3 100.1 mm to (-7.55, -33.8), turned to 180 degrees
- moved TP2 93.1 mm to (-7.50, 42.0)
- moved J11 91.9 mm to (-5.00, 26.6), turned to -90 degrees
- moved C7 90.6 mm to (2.25, 34.0), turned to -90 degrees
- moved J10 87.6 mm to (-5.00, 6.25), turned to -90 degrees
- moved J6 80.7 mm to (-38.0, 33.5), turned to 90 degrees
- moved TP3 77.2 mm to (-7.25, -41.2)
- moved J15 77.0 mm to (-32.0, -40.5), turned to 180 degrees
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- renumbered D2 to D1, D3 to D2, D4 to D3, D1 to D4
Connections:
- net /GND renamed GND
- J2 pad 4: /IO0 -> /IO1
Other:
- board text added: "3.3V+"
- board text added: "3V3_SENS"
- board text added: "5V0"
- board text added: "5V0+"
- board text added: "BNO085"
- board text added: "ESP32-S3"
- board text added: "GND"
- board text added: "MINI360"
- board text added: "MOTOR_L"
- board text added: "MOTOR_R"
- board text added: "MP1584EN"
- board text added: "TAU_1201"
- board text added: "VBAT_SK"
