File: UWB_ESP32S3_MainBoard_v2/UWB_ESP32S3_MainBoard_v2/UWB_ESP32S3_MainBoard_v2.kicad_sch (KiCad schematic)
At the start: 42 parts, among them J1 ESP32_S3_2, J10 MP1584EN_IN, J11 MP1584EN_OUT, J12 MINI360_IN, J13 MINI360_OUT, J14 VBAT, J15 MOTOR_L, J16 MOTOR_R, J2 ESP32_S3_1, J3 BNO085, J4 DRV8833_L_OUT, J5 DRV8833_L_IN, J6 DRV8833_R_OUT, J7 DRV8833_R_IN, J8 TAU_1201, J9 ESP32_UWBAOA_UART

Commit message: 테스트
Connections:
- net EEP: no longer J5.1 (Pin_1)
- net IO4: now also J8.3 (Pin_3); no longer J8.4 (Pin_4)
- net IO47: now also J3.4 (Pin_4); no longer J3.3 (Pin_3)
- net IO48: now also J3.3 (Pin_3); no longer J3.4 (Pin_4)
- net IO5: now also J8.4 (Pin_4); no longer J8.3 (Pin_3)
- net IO6: now also J9.5 (Pin_5); no longer J9.3 (Pin_3)
- net IO8: now also J9.3 (Pin_3); no longer J9.5 (Pin_5)
- net LF_A: now also J15.1 (Pin_1); no longer J15.4 (Pin_4)
- net LF_B: now also J15.2 (Pin_2); no longer J15.3 (Pin_3)
- net LR_A: now also J15.3 (Pin_3); no longer J15.2 (Pin_2)
- net LR_B: now also J15.4 (Pin_4); no longer J15.1 (Pin_1)
- net ULT: no longer J5.6 (Pin_6)
- no-connect marks 39 -> 40
Other:
- note added: "EEP"
- note added: "ULT"
- moved on the sheet: J15, J3
